File: soc_power_sch.kicad_sch (KiCad schematic)
At the start: 1 part, among them U1 AM6254ATCGHAALW

Commit message: commit++
Parts:
- removed U1: AM6254ATCGHAALW, pepy_sym_lib:[CPU]Texas Instruments AM6254ATCGHAALW, symbol pepy_sym_lib:[CPU]Texas Instruments AM6254ATCGHAALW
- added U1: AM6254ATCGHAALW, pepy_sym_lib:[CPU]Texas Instruments AM6254ATCGHAALW, symbol pepy_sym_lib:[CPU]Texas Instruments AM6254ATCGHAALW
Changed lines of the file:
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@@
 	(symbol
 		(lib_id "pepy_sym_lib:[CPU]Texas Instruments AM6254ATCGHAALW")
-		(at 41.91 101.6 0)
-		(unit 5)
+		(at 121.92 129.54 0)
+		(unit 2)
 		(exclude_from_sim no)
 		(in_bom yes)
@@
 		(fields_autoplaced yes)
 		(property "Reference" "U1"
-			(at 41.91 31.75 0)
+			(at 121.92 24.13 0)
 			(effects
 				(font
@@
 		)
 		(property "Value" "AM6254ATCGHAALW"
-			(at 41.91 34.29 0)
+			(at 121.92 26.67 0)
 			(effects
 				(font
@@
 		)
 		(property "Footprint" "pepy_sym_lib:[CPU]Texas Instruments AM6254ATCGHAALW"
-			(at 41.656 108.458 0)
+			(at 121.666 136.398 0)
 			(effects
 				(font
@@
 		)
 		(property "Datasheet" "https://www.ti.com/lit/ds/symlink/am625.pdf?ts=1740314582358&ref_url=https%253A%252F%252Fwww.ti.com%252Fmicrocontrollers-mcus-processors%252Farm-based-processors%252Fproducts.html"
-			(at 41.91 113.284 0)
+			(at 121.92 141.224 0)
 			(effects
 				(font
@@
 		)
 		(property "Description" "1400MHz FCCSP(ALW)-425 Microcontrollers (MCU/MPU/SOC) ROHS"
-			(at 41.656 115.57 0)
+			(at 121.666 143.51 0)
 			(effects
 				(font
@@
 		)
 		(property "LCSC Part" "C5218241"
-			(at 41.656 110.998 0)
+			(at 121.666 138.938 0)
 			(effects
 				(font
@@
 		)
 		(property "Manufacturer" "Texas Instruments"
-			(at 41.402 117.856 0)
+			(at 121.412 145.796 0)
 			(effects
 				(font
@@
 		(instances
 			(project "dashcam"
-				(path "/30d6913c-7aa4-4f56-9882-2ba08f7e2cce/0c9ede41-0025-44c0-8f9b-052975d40eea"
+				(path "/30d6913c-7aa4-4f56-9882-2ba08f7e2cce/9edd5e4e-bb8e-4c81-bbf2-addd01d032ef"
 					(reference "U1")
-					(unit 5)
+					(unit 2)
 				)
 			)

Commit message: PMIC draft
Connections:
- net VDD_CORE: now reaches U1.H8 (VDD_CORE)
- net VDD_CORE: now also U1.J11 (VDD_CORE), U1.J14 (VDD_CORE), U1.K17 (VDD_CORE), U1.L12 (VDD_CORE), U1.L15 (VDD_CORE), U1.M16 (VDD_CORE), U1.N11 (VDD_CORE), U1.N13 (VDD_CORE), U1.N8 (VDD_CORE), U1.P17 (VDD_CORE), U1.R11 (VDD_CORE), U1.R14 (VDD_CORE), U1.U12 (VDD_CORE), U1.V15 (VDD_CORE), U1.V17 (VDD_CORE), U1.V8 (VDD_CORE)
Other:
- note added: "Recommended operating conditions VDD_CORE: 0.715 0.75 0.79 [V]"
