File: usb_c.kicad_sch (KiCad schematic)
At the start: 12 parts, among them J1 TYPE-C 16PIN 2MD(073), U1 AM6254ATCGHAALW, U3 TVS0500DRVR

Commit message: SD card changes
Parts:
- renumbered R9 to R10, R8 to R11, R11 to R8, R10 to R9
Changed lines of the file:
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@@
 		(dnp no)
 		(fields_autoplaced yes)
-		(property "Reference" "R9"
+		(property "Reference" "R10"
 			(at 175.26 62.23 0)
 			(effects
@@
 			(project "dashcam"
 				(path "/30d6913c-7aa4-4f56-9882-2ba08f7e2cce/c5ef26fc-2066-490b-8721-1c4a1c83f953"
-					(reference "R9")
+					(reference "R10")
 					(unit 1)
 				)
@@
 		(on_board yes)
 		(dnp no)
-		(property "Reference" "#PWR06"
+		(property "Reference" "#PWR07"
 			(at 33.02 77.47 0)
 			(effects
@@
 			(project "dashcam"
 				(path "/30d6913c-7aa4-4f56-9882-2ba08f7e2cce/c5ef26fc-2066-490b-8721-1c4a1c83f953"
-					(reference "#PWR06")
+					(reference "#PWR07")
 					(unit 1)
 				)
@@
 		(dnp no)
 		(fields_autoplaced yes)
-		(property "Reference" "R11"
+		(property "Reference" "R8"
 			(at 154.94 53.3399 90)
 			(effects
@@
 			(project ""
 				(path "/30d6913c-7aa4-4f56-9882-2ba08f7e2cce/c5ef26fc-2066-490b-8721-1c4a1c83f953"
-					(reference "R11")
+					(reference "R8")
 					(unit 1)
 				)
@@
 		(on_board yes)
 		(dnp no)
-		(property "Reference" "#PWR08"
+		(property "Reference" "#PWR05"
 			(at 24.13 102.87 0)
 			(effects
@@
 			(project "dashcam"
 				(path "/30d6913c-7aa4-4f56-9882-2ba08f7e2cce/c5ef26fc-2066-490b-8721-1c4a1c83f953"
-					(reference "#PWR08")
+					(reference "#PWR05")
 					(unit 1)
 				)
@@
 		(on_board yes)
 		(dnp no)
-		(property "Reference" "#PWR09"
+		(property "Reference" "#PWR010"
 			(at 92.71 101.6 0)
 			(effects
@@
 			(project "dashcam"
 				(path "/30d6913c-7aa4-4f56-9882-2ba08f7e2cce/c5ef26fc-2066-490b-8721-1c4a1c83f953"
-					(reference "#PWR09")
+					(reference "#PWR010")
 					(unit 1)
 				)
@@
 		(on_board yes)
 		(dnp no)
-		(property "Reference" "#PWR010"
+		(property "Reference" "#PWR09"
 			(at 50.8 62.23 0)
 			(effects
@@
 			(project ""
 				(path "/30d6913c-7aa4-4f56-9882-2ba08f7e2cce/c5ef26fc-2066-490b-8721-1c4a1c83f953"
-					(reference "#PWR010")
+					(reference "#PWR09")
 					(unit 1)
 				)
@@
 		(dnp no)
 		(fields_autoplaced yes)
-		(property "Reference" "R8"
+		(property "Reference" "R11"
 			(at 181.61 97.7899 90)
 			(effects
@@
 			(project ""
 				(path "/30d6913c-7aa4-4f56-9882-2ba08f7e2cce/c5ef26fc-2066-490b-8721-1c4a1c83f953"
-					(reference "R8")
+					(reference "R11")
 					(unit 1)
 				)
@@
 		(on_board yes)
 		(dnp no)
-		(property "Reference" "#PWR07"
+		(property "Reference" "#PWR06"
 			(at 30.48 118.11 0)
 			(effects
@@
 			(project "dashcam"
 				(path "/30d6913c-7aa4-4f56-9882-2ba08f7e2cce/c5ef26fc-2066-490b-8721-1c4a1c83f953"
-					(reference "#PWR07")
+					(reference "#PWR06")
 					(unit 1)
 				)
@@
 		(on_board yes)
 		(dnp no)
-		(property "Reference" "#PWR05"
+		(property "Reference" "#PWR08"
 			(at 46.99 111.76 0)
 			(effects
@@
 			(project ""
 				(path "/30d6913c-7aa4-4f56-9882-2ba08f7e2cce/c5ef26fc-2066-490b-8721-1c4a1c83f953"
-					(reference "#PWR05")
+					(reference "#PWR08")
 					(unit 1)
 				)
@@
 		(dnp no)
 		(fields_autoplaced yes)
-		(property "Reference" "R10"
+		(property "Reference" "R9"
 			(at 154.94 63.4999 90)
 			(effects
@@
 			(project ""
 				(path "/30d6913c-7aa4-4f56-9882-2ba08f7e2cce/c5ef26fc-2066-490b-8721-1c4a1c83f953"
-					(reference "R10")
+					(reference "R9")
 					(unit 1)
 				)
@@
 		(on_board yes)
 		(dnp no)
-		(property "Reference" "#PWR011"
+		(property "Reference" "#PWR013"
 			(at 179.07 110.49 0)
 			(effects
@@
 			(project ""
 				(path "/30d6913c-7aa4-4f56-9882-2ba08f7e2cce/c5ef26fc-2066-490b-8721-1c4a1c83f953"
-					(reference "#PWR011")
+					(reference "#PWR013")
 					(unit 1)
 				)
@@
 		(on_board yes)
 		(dnp no)
-		(property "Reference" "#PWR013"
+		(property "Reference" "#PWR011"
 			(at 152.4 76.2 0)
 			(effects
@@
 			(project ""
 				(path "/30d6913c-7aa4-4f56-9882-2ba08f7e2cce/c5ef26fc-2066-490b-8721-1c4a1c83f953"
-					(reference "#PWR013")
+					(reference "#PWR011")
 					(unit 1)
 				)
