File: sd.kicad_sch (KiCad schematic)
At the start: 24 parts, among them U7 TPS22918DBVR

Commit message: Bulk change
Parts:
- added R82: RC0201FR-0733RL, pepy_sym_lib:[RES_SMD_0201_0603Metric], symbol pepy_sym_lib:[RES_SMD_0201_0603Metric]YAGEO RC0201FR-0733RL
- added R83: 0402WGF0000TCE, pepy_sym_lib:[RES_SMD_0402_1005Metric], symbol pepy_sym_lib:[RES_SMD_0402_1005Metric]UNI-ROYAL(Uniroyal Elec) 0402WGF0000TCE
- added U1: AM6254ATCGHAALW, pepy_sym_lib:[CPU]Texas Instruments AM6254ATCGHAALW, symbol pepy_sym_lib:[CPU]Texas Instruments AM6254ATCGHAALW
Connections:
- net SD_CD: now reaches R75.1
- net SD_CD: now also D9.2 (A), SD1.9 (CD), U1.D17 (MMC1_SDCD)
- net SD_CLK: now reaches R79.1
- net SD_CLK: now also D13.2 (A), SD1.5 (CLX), R83.2
- net VDD_SD: now reaches R79.2
- net VDD_SD: now also R76.2, R77.2, R78.2, R80.2, R81.2
- net SD_D1: now reaches R81.1
- net SD_D1: now also D15.2 (A), SD1.8 (DAT1), U1.B21 (MMC1_DAT1)
- net at D11.1 (C): now also D10.1 (C), D12.1 (C), D13.1 (C), D14.1 (C), D15.1 (C), D9.1 (C)
- net SD_D3: now reaches D11.2 (A)
- net SD_D3: now also R78.1, SD1.2 (CD/DAT3), U1.D22 (MMC1_DAT3)
- net SD_D0: now reaches D14.2 (A)
- net SD_D0: now also R80.1, SD1.7 (DAT0), U1.A22 (MMC1_DAT0)
- net SD_D2: now reaches SD1.1 (DAT2)
- net SD_D2: now also D10.2 (A), R76.1, U1.C21 (MMC1_DAT2)
- net SD_CMD: now reaches SD1.3 (CMD)
- net SD_CMD: now also D12.2 (A), R77.1, U1.A21 (MMC1_CMD)
- new net: R82.1, U1.D25 (MMC2_CLK)
- new net: R83.1, U1.B22 (MMC1_CLK)
- new net SD_VOLT_SEL: U1.C17 (MMC1_SDWP)
Other:
- moved on the sheet: C56, C57, C58, C59, C60, D10, D11, D12, D13, D14, D15, D7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
