File: hw/LTE.kicad_sch (KiCad schematic)
At the start: 90 parts, among them J10 IPX, J11 Host, J5 USB_OTG, J6 IPX, J7 Conn_01x04, J8 IPX, J9 IPX, P1 SK-C793, Q10 NMOS, Q3 NMOS, Q4 PMOS, Q5 NMOS, Q6 NMOS, Q7 NMOS, Q8 NMOS, Q9 NMOS, U12 M3406-ADJ, U13 sim7600, U14 USBLC6-2SC6, U15 74LVC1G80GV,125

Commit message: WIP SIM module
Parts:
- removed C166, C174, C181, C182, C192: 0.1uF 50v X5R, Capacitor_SMD:C_0603_1608Metric, symbol Device:C_Small
- removed C170, C175: 22uF 16v X5R, Capacitor_SMD:C_0805_2012Metric, symbol Device:C_Small
- removed C171, C172, C176, C177, C178: 1000uF 10v, Capacitor_THT:CP_Radial_D8.0mm_P3.50mm, symbol Device:CP_Small
- removed C173: 100pF C0G, Capacitor_SMD:C_0402_1005Metric, symbol Device:C_Small
- removed C179, C180: 1uF 16v X5R, Capacitor_SMD:C_0603_1608Metric, symbol Device:C_Small
- removed C186, C189, C191: 33pF C0G, Capacitor_SMD:C_0402_1005Metric, symbol Device:C_Small
- removed D24, D25: SS14, Diode_SMD:D_SMA, symbol Device:D_Schottky_Small_ALT
- removed D28, D29, D30: TVS, Diode_SMD:D_SOD-523, symbol Device:D_Zener_ALT
- removed J11: Host, cicada-footprints:PinSocket_2x08_P2.54mm_Vertical_padded, symbol connector:Conn_02x8_Odd_Even_Side_padding
- removed J5: USB_OTG, cicada-footprints:ZX62D-B-5PA8, symbol Connector:USB_OTG
- removed L12: LQG15HS1N0S02D, pepy_sym_lib:[IND_SMD_0402_1005Metric], symbol pepy_sym_lib:[IND_SMD_0402_1005Metric]Murata Electronics LQG15HS1N0S02D
- removed L13: MLG1005S0N5BT000, pepy_sym_lib:[IND_SMD_0402_1005Metric], symbol pepy_sym_lib:[IND_SMD_0402_1005Metric]TDK MLG1005S0N5BT000
- removed L8: 3.3uH 2A, cicada-footprints:L_4030_Handsoldering, symbol Device:L_Small
- removed P1: SK-C793, cicada-footprints:SK-C793, symbol SK-C793:SK-C793
- removed Q10, Q5, Q6, Q7, Q8, Q9: NMOS, Package_TO_SOT_SMD:SOT-23, symbol Device:Q_NMOS_GSD
- removed R122, R123: 40.2k, Resistor_SMD:R_0402_1005Metric, symbol Device:R_Small
- removed R124: 6.98k, Resistor_SMD:R_0402_1005Metric, symbol Device:R_Small
- removed R132, R133, R134: 22R, Resistor_SMD:R_0402_1005Metric, symbol Device:R_Small
- removed R135, R136, R137, R138, R139, R140, R141, R142, R143, R144, R145, R146: 4.7k, Resistor_SMD:R_0402_1005Metric, symbol Device:R_Small
- removed R147: 54.9k, Resistor_SMD:R_0402_1005Metric, symbol Device:R_Small
- removed R148: 340k, Resistor_SMD:R_0402_1005Metric, symbol Device:R_Small
- removed U12: M3406-ADJ, Package_TO_SOT_SMD:TSOT-23-5, symbol Regulator_Switching:LTC3406ES5
- removed unit 2 of U13
- removed U14: USBLC6-2SC6, Package_TO_SOT_SMD:SOT-23-6, symbol Power_Protection:USBLC6-2SC6
- removed U15: 74LVC1G80GV,125, pepy_sym_lib:[1CH_D_FLIP_FLOP]Nexperia 74LVC1G80GV,125, symbol pepy_sym_lib:[1CH_D_FLIP_FLOP]Nexperia 74LVC1G80GV,125
- added C189, C211, C214: CC1206KKX7RDBB102, pepy_sym_lib:[CAP_SMD_1206_3216Metric], symbol pepy_sym_lib:[CAP_SMD_1206_3216Metric]YAGEO CC1206KKX7RDBB102
- added C190, C191, C192, C193, C205, C206, C207, C208: CC0201KRX5R6BB104, pepy_sym_lib:[CAP_SMD_0201_0603Metric], symbol pepy_sym_lib:[CAP_SMD_0201_0603Metric]YAGEO CC0201KRX5R6BB104
- added C194, C195, C196, C197: GRM0335C1H100JA01D, pepy_sym_lib:[CAP_SMD_0201_0603Metric], symbol pepy_sym_lib:[CAP_SMD_0201_0603Metric]muRata GRM0335C1H100JA01D
- added C204: RVT1A331M0607, pepy_sym_lib:[CAP_SMD_AL_ELECTROLYTIC]ROQANG RVT1A331M0607, symbol pepy_sym_lib:[CAP_SMD_AL_ELECTROLYTIC]ROQANG RVT1A331M0607
- added C209, C210, C212, C213: CL31A107MQHNNNE, pepy_sym_lib:[CAP_SMD_1206_3216Metric], symbol pepy_sym_lib:[CAP_SMD_1206_3216Metric]Samsung Electro-Mechanics CL31A107MQHNNNE
- added C218, C219: GRM0335C1H470JA01D, pepy_sym_lib:[CAP_SMD_0201_0603Metric], symbol pepy_sym_lib:[CAP_SMD_0201_0603Metric]muRata GRM0335C1H470JA01D
- added C220, C221, C222: GRM0335C1H330JA01D, pepy_sym_lib:[CAP_SMD_0201_0603Metric], symbol pepy_sym_lib:[CAP_SMD_0201_0603Metric]muRata GRM0335C1H330JA01D
- added D29: ESD56151W05, pepy_sym_lib:[ESD_PROT]WILLSEMI ESD56151W05-2TR, symbol pepy_sym_lib:[ESD_PROT]WILLSEMI ESD56151W05-2TR
- added D30: LTST-C190KRKT, pepy_sym_lib:[LED]Lite-On LTST-C190KRKT, symbol pepy_sym_lib:[LED]Lite-On LTST-C190KRKT
- added D31: ESD56151W05-2/TR, pepy_sym_lib:[ESD_PROT]WILLSEMI ESD56151W05-2TR, symbol pepy_sym_lib:[ESD_PROT]WILLSEMI ESD56151W05-2TR
- added D32: ESDA6V1W5, pepy_sym_lib:[ESD_PROT]TECH PUBLIC ESDA6V1W5, symbol pepy_sym_lib:[ESD_PROT]TECH PUBLIC ESDA6V1W5
- added D33: USBLC6-2P6, pepy_sym_lib:[ESD_PROT]STMicroelectronics USBLC6-2P6, symbol pepy_sym_lib:[ESD_PROT]STMicroelectronics USBLC6-2P6
- added J11, J12, J16, J8, J9: U.FL-R-SMT-1(80), pepy_sym_lib:[SMD_COAXIAL_CONNECTOR]HRS(Hirose) U.FL-R-SMT-1(80), symbol pepy_sym_lib:[SMD_COAXIAL_CONNECTOR]HRS(Hirose) U.FL-R-SMT-1(80)
- added J17: USB-231-ARY, pepy_sym_lib:[USB_A_4P_RA_FEMALE]XUNPU USB-231-ARY, symbol pepy_sym_lib:[USB_A_4P_RA_FEMALE]XUNPU USB-231-ARY
- added J18: SMN-305-ARP7, pepy_sym_lib:[U_SIM]XUNPU SMN-305-ARP7, symbol pepy_sym_lib:[U_SIM]XUNPU SMN-305-ARP7
- added J6: S3B-ZR-SM4A-TF(LF)(SN), pepy_sym_lib:[JST_1X3P_1_5MM_R_ANGLE]JST S3B-ZR-SM4A-TF(LF)(SN), symbol pepy_sym_lib:[JST_1X3P_1_5MM_R_ANGLE]JST S3B-ZR-SM4A-TF(LF)(SN)
- added J7: PH2.54-01-03PZS, pepy_sym_lib:[2x3_PIN_HEADER_STR]XUNPU PH2.54-01-03PZS, symbol pepy_sym_lib:[2x3_PIN_HEADER_STR]XUNPU PH2.54-01-03PZS
- added L12, L13, L14: LQG15HS3N0S02D, pepy_sym_lib:[IND_SMD_0402_1005Metric], symbol pepy_sym_lib:[IND_SMD_0402_1005Metric]Murata Electronics LQG15HS3N0S02D
- added Q8: BSS138PW,115, pepy_sym_lib:[NMOS]Nexperia BSS138PW,115, symbol pepy_sym_lib:[NMOS]Nexperia BSS138PW,115
- added R164, R185, R191, R192: 0805W8F1004T5E, pepy_sym_lib:[RES_SMD_0805_2012Metric], symbol pepy_sym_lib:[RES_SMD_0805_2012Metric]UNI-ROYAL(Uniroyal Elec) 0805W8F1004T5E
- added R165, R180, R183: 0201WMF1002TEE, pepy_sym_lib:[RES_SMD_0201_0603Metric], symbol pepy_sym_lib:[RES_SMD_0201_0603Metric]UNI-ROYAL(Uniroyal Elec) 0201WMF1002TEE
- added R168, R169, R170, R171, R178, R179: 0402WGF0000TCE, pepy_sym_lib:[RES_SMD_0402_1005Metric], symbol pepy_sym_lib:[RES_SMD_0402_1005Metric]UNI-ROYAL(Uniroyal Elec) 0402WGF0000TCE
- added R177: RC0402FR-071KL, pepy_sym_lib:[RES_SMD_0402_1005Metric], symbol pepy_sym_lib:[RES_SMD_0402_1005Metric]YAGEO RC0402FR-071KL
- added R181: RC0402FR-07100KL, pepy_sym_lib:[RES_SMD_0402_1005Metric], symbol pepy_sym_lib:[RES_SMD_0402_1005Metric]YAGEO RC0402FR-07100KL
- added R182: 0402WGF4702TCE, pepy_sym_lib:[RES_SMD_0402_1005Metric], symbol pepy_sym_lib:[RES_SMD_0402_1005Metric]UNI-ROYAL 0402WGF4702TCE
- added R186: 0805W8F4700T5E, pepy_sym_lib:[RES_SMD_0805_2012Metric], symbol pepy_sym_lib:[RES_SMD_0805_2012Metric]UNI-ROYAL(Uniroyal Elec) 0805W8F4700T5E
- added R187: RC0603FR-0710RL, pepy_sym_lib:[RES_SMD_0603_1608Metric], symbol pepy_sym_lib:[RES_SMD_0603_1608Metric]YAGEO RC0603FR-0710RL
- added R188, R193, R194: RC0201FR-0733RL, pepy_sym_lib:[RES_SMD_0201_0603Metric], symbol pepy_sym_lib:[RES_SMD_0201_0603Metric]YAGEO RC0201FR-0733RL
- added S1: TS-1088-AR02016, pepy_sym_lib:[TACTILE_SWITCH]XUNPU TS-1088-AR02016, symbol pepy_sym_lib:[TACTILE_SWITCH]XUNPU TS-1088-AR02016
- added TP19: DCD, symbol Connector:TestPoint
- added TP20: RI, symbol Connector:TestPoint
- added TP21: DTR, symbol Connector:TestPoint
- added TP22: RTS, symbol Connector:TestPoint
- added TP23: CTS, symbol Connector:TestPoint
- added TP24: SIM_STAT, symbol Connector:TestPoint
- added U12: TXU0202DCUR, pepy_sym_lib:[LEVEL_SHIFTER]TI TXU0202DCUR, symbol pepy_sym_lib:[LEVEL_SHIFTER]TI TXU0202DCUR
- added U14: TCA9406DCUR, pepy_sym_lib:[LEVEL_SHIFTER]TI TCA9406DCUR, symbol pepy_sym_lib:[LEVEL_SHIFTER]TI TCA9406DCUR
- added U15: SIM7600E, pepy_sym_lib:[GSM_3G_LTE]SIMCom Wireless Solutions SIM7600E, symbol pepy_sym_lib:[GSM_3G_LTE]SIMCom Wireless Solutions SIM7600E
- added U16: MIC29302WU, pepy_sym_lib:[LDO]MICROCHIP MIC29302WU-TR, symbol pepy_sym_lib:[LDO]MICROCHIP MIC29302WU-TR
- renumbered C183 to C198, C184 to C199, C185 to C200, C187 to C201, C188 to C202, C190 to C203, D20 to D23, D21 to D24, D22 to D25, D23 to D26, D26 to D27, D27 to D28, J6 to J10, J8 to J13, J9 to J14, J10 to J15, J7 to J5, Q3 to Q5, Q4 to Q6, R125 to R166, R126 to R167, R127 to R172, R128 to R173, R129 to R174, R130 to R175, R131 to R176, TP16 to TP17, TP17 to TP18
Connections:
- net AUX_ANT: now also J9.1
- net GND: now also C189.2, C190.1, C191.1, C192.2, C193.2, C194.1, C195.1, C196.1, C197.1, C204.2, C205.1, C206.1, C207.1, C208.1, C209.1, C210.1, C211.2, C212.1, C213.1, C214.2, C220.1, C221.1, C222.1, D29.1 (C), D31.1 (C), D32.2 (GND), D33.2 (GND), J11.2, J12.2, J16.2, J17.4 (GND), J18.5 (GND), J6.2, J8.2, J9.2, L12.1, L13.1, Q8.2 (S), R164.2, R182.1, R183.1, R185.1, R191.2, R192.2, U12.2 (GND), U14.2 (GND), U15.1 (GND), U15.10 (GND), U15.14 (GND), U15.2 (GND), U15.3 (PWRKEY), U15.37 (GND), U15.40 (GND), U15.41 (GND), U15.43 (GND), U15.5 (GND), U15.57 (GND), U15.58 (GND), U15.60 (GND), U15.61 (GND), U15.64 (GND), U15.65 (GND), U15.77 (GND), U15.78 (GND), U15.80 (GND), U15.81 (GND), U16.3 (GND), U16.6 (TAB)
- net GNSS_ANT: now also C219.1, L12.2
- net MAIN_ANT: now also J8.1
- net SIM_CLK: now also C221.2, D32.4, J18.3 (CLK), R194.1
- net SIM_RST: now also C220.2, D32.5, J18.2 (RST), R193.1
- net SIM_VCC: now also C206.2, D32.3, J18.1 (VCC), R187.2, U15.20 (USIM_VDD)
- net VBUS: now also D33.5 (VBUS), J17.1 (VBUS), U15.11 (USB_VBUS)
- net nRST: now also U15.4 (RESET)
- new net: C195.2, J9.1, R169.1
- new net: R177.1, U15.54 (FLIGHTMODE)
- new net: R180.1, S1.2
- new net: R165.2, U14.6 (OE)
- new net: TP22.1, U15.66 (RTS)
- new net: C196.2, R168.2, R170.1
- new net: C218.2, J16.1, L14.1
- new net: R181.1, R182.2, U16.5 (ADJ)
- new net: J11.1, R170.2
- new net: TP19.1, U15.70 (DCD)
- new net: C194.2, J8.1, R168.1
- new net: C197.2, R169.2, R171.1
- new net: J12.1, R171.2
- new net: C218.1, C219.2, L13.2
- new net: TP21.1, U15.72 (DTR)
- new net: R178.2, R179.2, U16.1 (EN)
- new net: D29.2 (A), S1.1, U15.85 (USB_BOOT)
- new net: L14.2, R187.1
- new net: D30.1 (A), R186.1
- new net: TP20.1, U15.69 (RI)
- new net: R193.2, U15.18 (USIM_RST)
- new net: R194.2, U15.19 (USIM_CLK)
- new net: D30.2 (C), Q8.3 (D)
- new net: R188.2, U15.17 (USIM_DATA)
- new net: TP24.1, U15.49 (STATUS)
- new net: TP23.1, U15.67 (CTS)
- new net 1V8_COMM: C191.2, C192.1, R165.1, R177.2, R180.2, U12.7 (VCCB), U14.3 (VCCA), U15.15 (VDD_1V8)
- new net BARREL_JACK: R178.1, U16.2 (VIN)
- new net COMM_SCL: U14.5 (SCL_A), U15.55 (SCL)
- new net COMM_SDA: U14.4 (SDA_A), U15.56 (SDA)
- new net D+: D33.1 (I/O1), D33.6 (I/O1), J17.3 (D+), U15.13 (USB_DP)
- new net D-: D33.3 (I/O2), D33.4 (I/O2), J17.2 (D-), U15.12 (USB_DN)
- new net EN: R179.1
- new net Earth: C211.1, J17.5 (Shield), J17.6 (Shield), R191.1
- new net Earth_SIM: C214.1, J18.10 (SH), J18.11 (SH), J18.8 (SH), J18.9 (SH), R192.1
- new net Earth_UART_CONN: C189.1, J6.4, J6.5, R164.1
- new net M_RX_S_TX: J7.4, U12.4 (A2Y)
- new net M_RX_S_TX_1V8: U12.1 (B2), U15.71 (TXD)
- new net M_RX_S_TX_HOST: J7.2
- new net M_RX_S_TX_OUT: J6.3, J7.6
- new net M_TX_S_RX: J7.3, U12.5 (A1)
- new net M_TX_S_RX_1V8: U12.8 (B1Y), U15.68 (RXD)
- new net M_TX_S_RX_HOST: J7.1
- new net M_TX_S_RX_OUT: J6.1, J7.5
- new net NETFLIGHT: Q8.1 (G), R183.2, R185.2
- new net NETLIGHT: U15.51 (NETLIGHT)
- new net SCL: U14.8 (SCL_B)
- new net SDA: U14.1 (SDA_B)
- new net SIM_DATA: C222.2, D32.1, J18.7 (I/O), R188.1
- new net VDD_3V3: C190.2, C193.1, R186.2, U12.3 (VCCA), U12.6 (OE), U14.7 (VCCB)
- new net VDD_COMM: C204.1, C205.2, C207.2, C208.2, C209.2, C210.2, C212.2, C213.2, D31.2 (A), R181.2, U15.38 (VBAT), U15.39 (VBAT), U15.62 (VBAT), U15.63 (VBAT), U16.4 (VOUT)
- no-connect marks 42 -> 77
Other:
- note added: "90 Ohm"
- note added: "Always On Status: Searching Network; Call Connect (includes VOLTE, SRLTE) 200ms ON, 200ms OFF Status: Data Transmit; 4G registered 800ms ON, 800ms OFF Status: 2G/3G registered network OFF Status: Power off; Sleep"
- note added: "Flightmode:If unused keep it open or pull it to high."
- note added: "I2C"
- note added: "In case for some reason NETFLIGHT would be high when SIM is off. 10k pull down would do the trick. (That would "zero out" 1M.)"
- note added: "Netflight status"
- note added: "Note: M->Master S->Slave"
- note added: "Parasitic capacitance should not exceed 60pF."
- note added: "Place the bypass capacitors close (after ESD protection diodes) to the SIM card holder on all signals for improving EMI."
- note added: "Power on/off is realized through the LDO EN/DIS."
- note added: "RESET pin has been pulled up internally with a 40kOHm resistor to 1V8, hence no need to do so externally."
- note added: "SIM card"
- note added: "The TCA9406 device has 10kΩ internal pullup resistors. External pullup resistors can be added to reduce the total RC of a signal trace if necessary."
- note added: "USIM_DATA has been pulled up with a 10kΩ resistor to USIM_VDD in the module."
- note removed: "(Optional, for FW update)"
- note removed: "0"
- note removed: "1"
- note removed: "2"
- note removed: "2G"
- note removed: "3"
- note removed: "4"
- note removed: "4G"
- note removed: "5"
- note removed: "6"
- note removed: "7"
- note removed: "8"
- note removed: "9"
- note removed: "Datasheet suggests 10uF"
- note removed: "Datasheet suggests 4.7uF"
- note removed: "Dev"
- note removed: "Level shifters 1.8v <-> 3.3v"
- note removed: "Maj version"
- note removed: "Power supply"
- note removed: "The version resistor forms a voltage divider with a 40.2K resistor on the host board. The host then can read the version as an analog voltage value. Check out the table."
- note removed: "USB"
- note removed: "USIM Card"
- note removed: "VER_1 = 4"
- note removed: "VER_2 = 2"
- note removed: "Vout = 0.6 * (R1 + R2) / R2 Vout = 0.6 * (40.2 + 6.98) / 6.98 Vout = 4.06"
- note removed: "Vth < 1.8v"
- note removed: "WiFi"
- note removed: "~0.2R copper trace snaky. We want to prevent current spikes from propagating to the host side. Snake is more robust than a resistor, think hot-plug inrush current."
