File: hw/bootstrap.kicad_sch (KiCad schematic)
At the start: 39 parts

Commit message: WIP SIM module
Parts:
- renumbered R18 to R27, R19 to R28, R20 to R29, R21 to R30, R22 to R31, R23 to R32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
