File: hw/camera.kicad_sch (KiCad schematic)
At the start: 12 parts, among them J2 FPC-05F-22PH20, Q1 BSS138PW,115, Q2 BSS138PW,115, U1 AM6254ATCGHAALW

Commit message: WIP SIM module
Parts:
- renumbered C6 to C8, C7 to C9, J2 to J3, R12 to R21, R13 to R22, R14 to R23, R15 to R24, R16 to R25, R17 to R26
Changed lines of the file:
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@@
 		(dnp no)
 		(fields_autoplaced yes)
-		(property "Reference" "#PWR014"
+		(property "Reference" "#PWR018"
 			(at 62.23 38.1 0)
 			(effects
@@
 			(project ""
 				(path "/30d6913c-7aa4-4f56-9882-2ba08f7e2cce/0111536d-88df-4dfc-a217-9c0dd361d8c8"
-					(reference "#PWR014")
+					(reference "#PWR018")
 					(unit 1)
 				)
@@
 		(dnp no)
 		(fields_autoplaced yes)
-		(property "Reference" "R15"
+		(property "Reference" "R24"
 			(at 156.21 29.2099 90)
 			(effects
@@
 			(project "dashcam"
 				(path "/30d6913c-7aa4-4f56-9882-2ba08f7e2cce/0111536d-88df-4dfc-a217-9c0dd361d8c8"
-					(reference "R15")
+					(reference "R24")
 					(unit 1)
 				)
@@
 		(dnp no)
 		(fields_autoplaced yes)
-		(property "Reference" "J2"
+		(property "Reference" "J3"
 			(at 53.34 77.4699 0)
 			(effects
@@
 			(project ""
 				(path "/30d6913c-7aa4-4f56-9882-2ba08f7e2cce/0111536d-88df-4dfc-a217-9c0dd361d8c8"
-					(reference "J2")
+					(reference "J3")
 					(unit 1)
 				)
@@
 		(dnp no)
 		(fields_autoplaced yes)
-		(property "Reference" "C6"
+		(property "Reference" "C8"
 			(at 58.42 29.2101 90)
 			(effects
@@
 			(project ""
 				(path "/30d6913c-7aa4-4f56-9882-2ba08f7e2cce/0111536d-88df-4dfc-a217-9c0dd361d8c8"
-					(reference "C6")
+					(reference "C8")
 					(unit 1)
 				)
@@
 		(dnp no)
 		(fields_autoplaced yes)
-		(property "Reference" "R17"
+		(property "Reference" "R26"
 			(at 180.34 99.0599 90)
 			(effects
@@
 			(project ""
 				(path "/30d6913c-7aa4-4f56-9882-2ba08f7e2cce/0111536d-88df-4dfc-a217-9c0dd361d8c8"
-					(reference "R17")
+					(reference "R26")
 					(unit 1)
 				)
@@
 		(dnp no)
 		(fields_autoplaced yes)
-		(property "Reference" "R14"
+		(property "Reference" "R23"
 			(at 133.35 27.9399 90)
 			(effects
@@
 			(project ""
 				(path "/30d6913c-7aa4-4f56-9882-2ba08f7e2cce/0111536d-88df-4dfc-a217-9c0dd361d8c8"
-					(reference "R14")
+					(reference "R23")
 					(unit 1)
 				)
@@
 		(on_board yes)
 		(dnp no)
-		(property "Reference" "R12"
+		(property "Reference" "R21"
 			(at 76.2 58.42 0)
 			(effects
@@
 			(project ""
 				(path "/30d6913c-7aa4-4f56-9882-2ba08f7e2cce/0111536d-88df-4dfc-a217-9c0dd361d8c8"
-					(reference "R12")
+					(reference "R21")
 					(unit 1)
 				)
@@
 		(on_board yes)
 		(dnp no)
-		(property "Reference" "#PWR015"
+		(property "Reference" "#PWR019"
 			(at 68.58 116.84 0)
 			(effects
@@
 			(project ""
 				(path "/30d6913c-7aa4-4f56-9882-2ba08f7e2cce/0111536d-88df-4dfc-a217-9c0dd361d8c8"
-					(reference "#PWR015")
+					(reference "#PWR019")
 					(unit 1)
 				)
@@
 		(dnp no)
 		(fields_autoplaced yes)
-		(property "Reference" "R16"
+		(property "Reference" "R25"
 			(at 173.99 29.2099 90)
 			(effects
@@
 			(project "dashcam"
 				(path "/30d6913c-7aa4-4f56-9882-2ba08f7e2cce/0111536d-88df-4dfc-a217-9c0dd361d8c8"
-					(reference "R16")
+					(reference "R25")
 					(unit 1)
 				)
@@
 		(dnp no)
 		(fields_autoplaced yes)
-		(property "Reference" "R13"
+		(property "Reference" "R22"
 			(at 115.57 29.2099 90)
 			(effects
@@
 			(project ""
 				(path "/30d6913c-7aa4-4f56-9882-2ba08f7e2cce/0111536d-88df-4dfc-a217-9c0dd361d8c8"
-					(reference "R13")
+					(reference "R22")
 					(unit 1)
 				)
@@
 		(on_board yes)
 		(dnp no)
-		(property "Reference" "#PWR016"
+		(property "Reference" "#PWR020"
 			(at 177.8 111.76 0)
 			(effects
@@
 			(project ""
 				(path "/30d6913c-7aa4-4f56-9882-2ba08f7e2cce/0111536d-88df-4dfc-a217-9c0dd361d8c8"
-					(reference "#PWR016")
+					(reference "#PWR020")
 					(unit 1)
 				)
@@
 		(on_board yes)
 		(dnp no)
-		(property "Reference" "C7"
+		(property "Reference" "C9"
 			(at 71.882 29.718 90)
 			(effects
@@
 			(project ""
 				(path "/30d6913c-7aa4-4f56-9882-2ba08f7e2cce/0111536d-88df-4dfc-a217-9c0dd361d8c8"
-					(reference "C7")
+					(reference "C9")
 					(unit 1)
 				)
