File: hw/dcaps.kicad_sch (KiCad schematic)
At the start: 29 parts, among them U1 AM6254ATCGHAALW

Commit message: Ethernet...
Parts:
- added C100, C99: CC0402MRX5R5BB106, pepy_sym_lib:[CAP_SMD_0402_1005Metric], symbol pepy_sym_lib:[CAP_SMD_0402_1005Metric]YAGEO CC0402MRX5R5BB106
- added C101, C111, C119, C133: CL05A475KP5NRNC, pepy_sym_lib:[CAP_SMD_0402_1005Metric], symbol pepy_sym_lib:[CAP_SMD_0402_1005Metric]Samsung Electro-Mechanics CL05A475KP5NRNC
- added C102, C103, C104, C105, C106, C107, C108, C109, C110, C112, C113, C114, C115, C116, C117, C118, C120, C122, C123, C124, C125, C126, C127, C128, C129, C131, C135, C136, C137, C138, C139: CC0201KRX5R6BB104, pepy_sym_lib:[CAP_SMD_0201_0603Metric], symbol pepy_sym_lib:[CAP_SMD_0201_0603Metric]YAGEO CC0201KRX5R6BB104
- added C121, C130, C132: CL03A105MQ3CSNH, pepy_sym_lib:[CAP_SMD_0201_0603Metric], symbol pepy_sym_lib:[CAP_SMD_0201_0603Metric]Samsung Electro-Mechanics CL03A105MQ3CSNH
Connections:
- net GND: now also C100.1, C101.1, C102.1, C103.1, C104.1, C105.1, C106.1, C107.1, C108.1, C109.1, C110.1, C111.1, C112.1, C113.1, C114.1, C115.1, C116.1, C117.1, C118.1, C119.1, C120.1, C121.1, C122.1, C123.1, C124.1, C125.1, C126.1, C127.1, C128.1, C129.1, C130.1, C131.1, C132.1, C133.1, C135.1, C136.1, C137.1, C138.1, C139.1, C99.1
- new net VDDA_0V85: C101.2, C102.2, C103.2, C104.2, C105.2, C106.2, C107.2, C108.2, C109.2, C110.2, C99.2
- new net VDD_1V2: C100.2, C132.2, C133.2, C135.2, C136.2, C137.2, C138.2, C139.2
- new net VDD_1V8: C119.2, C120.2, C122.2, C123.2, C124.2, C125.2, C126.2, C127.2, C128.2, C129.2, C130.2, C131.2
- new net VDD_3V3: C111.2, C112.2, C113.2, C114.2, C115.2, C116.2, C117.2, C118.2, C121.2

Commit message: WIP SIM module
Parts:
- renumbered C8 to C10, C99 to C11, C121 to C12, C130 to C13, C132 to C14, C9 to C15, C101 to C16, C111 to C17, C119 to C18, C133 to C19, C10 to C20, C11 to C21, C102 to C22, C112 to C23, C120 to C24, C100 to C25, C12 to C26, C103 to C27, C113 to C28, C122 to C29, C135 to C30, C13 to C31, C104 to C32, C114 to C33, C123 to C34, C136 to C35, C14 to C36, C105 to C37, C115 to C38, C124 to C39, C137 to C40, C15 to C41, C106 to C42, C116 to C43, C125 to C44, C138 to C45, C16 to C46, C107 to C47, C117 to C48, C126 to C49, C139 to C50, C17 to C51, C108 to C52, C118 to C53, C127 to C54, C18 to C55, C109 to C56, C128 to C57, C19 to C58, C110 to C59, C129 to C60, C20 to C61, C131 to C62, C21 to C63, C22 to C64, C23 to C65, C24 to C66, C25 to C67, C26 to C68, C27 to C69, C28 to C70, C29 to C71, C30 to C72, C31 to C73, C32 to C74, C33 to C75, C34 to C76, C35 to C77
