File: hw/ddr.kicad_sch (KiCad schematic)
At the start: 44 parts, among them U1 AM6254ATCGHAALW, U11 K4AAG165WA-BCWE

Commit message: WIP SIM module
Parts:
- renumbered C149 to C156, C144 to C157, C150 to C158, C145 to C159, C151 to C160, C134 to C161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
