File: hw/display.kicad_sch (KiCad schematic)
At the start: 15 parts, among them J4 0.5K-DX-40PWB, U1 AM6254ATCGHAALW

Commit message: WIP SIM module
Parts:
- renumbered C61 to C1, C62 to C2, FB3 to FB1, J4 to J1, L7 to L1, L6 to L2, R87 to R2, R86 to R3, R85 to R4, R84 to R5, R88 to R6, R89 to R7, R90 to R8, R91 to R9
Changed lines of the file:
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@@
 		(dnp yes)
 		(fields_autoplaced yes)
-		(property "Reference" "R88"
+		(property "Reference" "R6"
 			(at 179.07 123.1899 90)
 			(effects
@@
 			(project ""
 				(path "/30d6913c-7aa4-4f56-9882-2ba08f7e2cce/0c9ede41-0025-44c0-8f9b-052975d40eea"
-					(reference "R88")
+					(reference "R6")
 					(unit 1)
 				)
@@
 		(on_board yes)
 		(dnp no)
-		(property "Reference" "#PWR062"
+		(property "Reference" "#PWR02"
 			(at 226.06 149.86 0)
 			(effects
@@
 			(project "dashcam"
 				(path "/30d6913c-7aa4-4f56-9882-2ba08f7e2cce/0c9ede41-0025-44c0-8f9b-052975d40eea"
-					(reference "#PWR062")
+					(reference "#PWR02")
 					(unit 1)
 				)
@@
 		(dnp no)
 		(fields_autoplaced yes)
-		(property "Reference" "L6"
+		(property "Reference" "L2"
 			(at 92.71 120.65 0)
 			(effects
@@
 			(project ""
 				(path "/30d6913c-7aa4-4f56-9882-2ba08f7e2cce/0c9ede41-0025-44c0-8f9b-052975d40eea"
-					(reference "L6")
+					(reference "L2")
 					(unit 1)
 				)
@@
 		(dnp no)
 		(fields_autoplaced yes)
-		(property "Reference" "FB3"
+		(property "Reference" "FB1"
 			(at 218.44 129.54 0)
 			(effects
@@
 			(project ""
 				(path "/30d6913c-7aa4-4f56-9882-2ba08f7e2cce/0c9ede41-0025-44c0-8f9b-052975d40eea"
-					(reference "FB3")
+					(reference "FB1")
 					(unit 1)
 				)
@@
 		(on_board yes)
 		(dnp no)
-		(property "Reference" "#PWR061"
+		(property "Reference" "#PWR03"
 			(at 254 25.4 0)
 			(effects
@@
 			(project "dashcam"
 				(path "/30d6913c-7aa4-4f56-9882-2ba08f7e2cce/0c9ede41-0025-44c0-8f9b-052975d40eea"
-					(reference "#PWR061")
+					(reference "#PWR03")
 					(unit 1)
 				)
@@
 		(dnp no)
 		(fields_autoplaced yes)
-		(property "Reference" "J4"
+		(property "Reference" "J1"
 			(at 260.35 76.1999 0)
 			(effects
@@
 			(project ""
 				(path "/30d6913c-7aa4-4f56-9882-2ba08f7e2cce/0c9ede41-0025-44c0-8f9b-052975d40eea"
-					(reference "J4")
+					(reference "J1")
 					(unit 1)
 				)
@@
 		(on_board yes)
 		(dnp no)
-		(property "Reference" "C61"
+		(property "Reference" "C1"
 			(at 226.822 137.922 90)
 			(effects
@@
 			(project ""
 				(path "/30d6913c-7aa4-4f56-9882-2ba08f7e2cce/0c9ede41-0025-44c0-8f9b-052975d40eea"
-					(reference "C61")
+					(reference "C1")
 					(unit 1)
 				)
@@
 		(dnp no)
 		(fields_autoplaced yes)
-		(property "Reference" "L7"
+		(property "Reference" "L1"
 			(at 92.71 88.9 0)
 			(effects
@@
 			(project "dashcam"
 				(path "/30d6913c-7aa4-4f56-9882-2ba08f7e2cce/0c9ede41-0025-44c0-8f9b-052975d40eea"
-					(reference "L7")
+					(reference "L1")
 					(unit 1)
 				)
@@
 		(on_board yes)
 		(dnp yes)
-		(property "Reference" "R84"
+		(property "Reference" "R5"
 			(at 92.71 139.7 0)
 			(effects
@@
 			(project ""
 				(path "/30d6913c-7aa4-4f56-9882-2ba08f7e2cce/0c9ede41-0025-44c0-8f9b-052975d40eea"
-					(reference "R84")
+					(reference "R5")
 					(unit 1)
 				)
@@
 		(on_board yes)
 		(dnp no)
-		(property "Reference" "#PWR060"
+		(property "Reference" "#PWR04"
 			(at 257.81 142.24 0)
 			(effects
@@
 			(project ""
 				(path "/30d6913c-7aa4-4f56-9882-2ba08f7e2cce/0c9ede41-0025-44c0-8f9b-052975d40eea"
-					(reference "#PWR060")
+					(reference "#PWR04")
 					(unit 1)
 				)
@@
 		(on_board yes)
 		(dnp no)
-		(property "Reference" "R87"
+		(property "Reference" "R2"
 			(at 92.71 83.82 0)
 			(effects
@@
 			(project "dashcam"
 				(path "/30d6913c-7aa4-4f56-9882-2ba08f7e2cce/0c9ede41-0025-44c0-8f9b-052975d40eea"
-					(reference "R87")
+					(reference "R2")
 					(unit 1)
 				)
@@
 		(dnp no)
 		(fields_autoplaced yes)
-		(property "Reference" "R89"
+		(property "Reference" "R7"
 			(at 186.69 123.1899 90)
 			(effects
@@
 			(project "dashcam"
 				(path "/30d6913c-7aa4-4f56-9882-2ba08f7e2cce/0c9ede41-0025-44c0-8f9b-052975d40eea"
-					(reference "R89")
+					(reference "R7")
 					(unit 1)
 				)
@@
 		(dnp no)
 		(fields_autoplaced yes)
-		(property "Reference" "C62"
+		(property "Reference" "C2"
 			(at 241.3 138.4299 90)
 			(effects
@@
 			(project ""
 				(path "/30d6913c-7aa4-4f56-9882-2ba08f7e2cce/0c9ede41-0025-44c0-8f9b-052975d40eea"
-					(reference "C62")
+					(reference "C2")
 					(unit 1)
 				)
@@
 		(on_board yes)
 		(dnp no)
-		(property "Reference" "#PWR063"
+		(property "Reference" "#PWR01"
 			(at 176.53 135.89 0)
 			(effects
@@
 			(project "dashcam"
 				(path "/30d6913c-7aa4-4f56-9882-2ba08f7e2cce/0c9ede41-0025-44c0-8f9b-052975d40eea"
-					(reference "#PWR063")
+					(reference "#PWR01")
 					(unit 1)
 				)
@@
 		(on_board yes)
 		(dnp no)
-		(property "Reference" "R86"
+		(property "Reference" "R3"
 			(at 92.71 104.14 0)
 			(effects
@@
 			(project "dashcam"
 				(path "/30d6913c-7aa4-4f56-9882-2ba08f7e2cce/0c9ede41-0025-44c0-8f9b-052975d40eea"
-					(reference "R86")
+					(reference "R3")
 					(unit 1)
 				)
@@
 		(on_board yes)
 		(dnp yes)
-		(property "Reference" "R85"
+		(property "Reference" "R4"
 			(at 92.71 113.03 0)
 			(effects
@@
 			(project "dashcam"
 				(path "/30d6913c-7aa4-4f56-9882-2ba08f7e2cce/0c9ede41-0025-44c0-8f9b-052975d40eea"
-					(reference "R85")
+					(reference "R4")
 					(unit 1)
 				)
@@
 		(dnp no)
 		(fields_autoplaced yes)
-		(property "Reference" "R90"
+		(property "Reference" "R8"
 			(at 195.58 123.1899 90)
 			(effects
@@
 			(project "dashcam"
 				(path "/30d6913c-7aa4-4f56-9882-2ba08f7e2cce/0c9ede41-0025-44c0-8f9b-052975d40eea"
-					(reference "R90")
+					(reference "R8")
 					(unit 1)
 				)
@@
 		(dnp no)
 		(fields_autoplaced yes)
-		(property "Reference" "R91"
+		(property "Reference" "R9"
 			(at 204.47 123.1899 90)
 			(effects
@@
 			(project "dashcam"
 				(path "/30d6913c-7aa4-4f56-9882-2ba08f7e2cce/0c9ede41-0025-44c0-8f9b-052975d40eea"
-					(reference "R91")
-					(unit 1)
-				)
+					(reference "R9")
+					(unit 1)
+				)
