File: hw/eeprom.kicad_sch (KiCad schematic)
At the start: 4 parts

Commit message: eMMC draft
Parts:
- gave numbers to parts that had none: 3
Changed lines of the file:
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@@
 		(dnp no)
 		(fields_autoplaced yes)
-		(property "Reference" "R?"
+		(property "Reference" "R95"
 			(at 63.5 68.5799 90)
 			(effects
@@
 			(project "dashcam"
 				(path "/30d6913c-7aa4-4f56-9882-2ba08f7e2cce/e32d7694-9c48-497a-b173-43968d858b60"
-					(reference "R?")
+					(reference "R95")
 					(unit 1)
 				)
@@
 		(dnp no)
 		(fields_autoplaced yes)
-		(property "Reference" "C?"
+		(property "Reference" "C66"
 			(at 62.23 41.9099 90)
 			(effects
@@
 			(project "dashcam"
 				(path "/30d6913c-7aa4-4f56-9882-2ba08f7e2cce/e32d7694-9c48-497a-b173-43968d858b60"
-					(reference "C?")
+					(reference "C66")
 					(unit 1)
 				)
@@
 		(on_board yes)
 		(dnp no)
-		(property "Reference" "#PWR?"
+		(property "Reference" "#PWR064"
 			(at 77.47 53.34 0)
 			(effects
@@
 			(project "dashcam"
 				(path "/30d6913c-7aa4-4f56-9882-2ba08f7e2cce/e32d7694-9c48-497a-b173-43968d858b60"
-					(reference "#PWR?")
+					(reference "#PWR064")
 					(unit 1)
 				)
@@
 		(dnp no)
 		(fields_autoplaced yes)
-		(property "Reference" "U?"
+		(property "Reference" "U8"
 			(at 86.36 33.02 0)
 			(effects
@@
 			(project "dashcam"
 				(path "/30d6913c-7aa4-4f56-9882-2ba08f7e2cce/e32d7694-9c48-497a-b173-43968d858b60"
-					(reference "U?")
+					(reference "U8")
 					(unit 1)
 				)

Commit message: WIP SIM module
Parts:
- renumbered C66 to C155, R95 to R150, R93 to R151, U8 to U9
Changed lines of the file:
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@@
 		(dnp no)
 		(fields_autoplaced yes)
-		(property "Reference" "R95"
+		(property "Reference" "R150"
 			(at 63.5 68.5799 90)
 			(effects
@@
 			(project "dashcam"
 				(path "/30d6913c-7aa4-4f56-9882-2ba08f7e2cce/e32d7694-9c48-497a-b173-43968d858b60"
-					(reference "R95")
+					(reference "R150")
 					(unit 1)
 				)
@@
 		(dnp no)
 		(fields_autoplaced yes)
-		(property "Reference" "C66"
+		(property "Reference" "C155"
 			(at 62.23 41.9099 90)
 			(effects
@@
 			(project "dashcam"
 				(path "/30d6913c-7aa4-4f56-9882-2ba08f7e2cce/e32d7694-9c48-497a-b173-43968d858b60"
-					(reference "C66")
+					(reference "C155")
 					(unit 1)
 				)
@@
 		(on_board yes)
 		(dnp no)
-		(property "Reference" "#PWR065"
+		(property "Reference" "#PWR0108"
 			(at 60.96 91.44 0)
 			(effects
@@
 			(project "dashcam"
 				(path "/30d6913c-7aa4-4f56-9882-2ba08f7e2cce/e32d7694-9c48-497a-b173-43968d858b60"
-					(reference "#PWR065")
+					(reference "#PWR0108")
 					(unit 1)
 				)
@@
 		(on_board yes)
 		(dnp no)
-		(property "Reference" "#PWR064"
+		(property "Reference" "#PWR0109"
 			(at 77.47 53.34 0)
 			(effects
@@
 			(project "dashcam"
 				(path "/30d6913c-7aa4-4f56-9882-2ba08f7e2cce/e32d7694-9c48-497a-b173-43968d858b60"
-					(reference "#PWR064")
+					(reference "#PWR0109")
 					(unit 1)
 				)
@@
 		(dnp no)
 		(fields_autoplaced yes)
-		(property "Reference" "U8"
+		(property "Reference" "U9"
 			(at 86.36 33.02 0)
 			(effects
@@
 			(project "dashcam"
 				(path "/30d6913c-7aa4-4f56-9882-2ba08f7e2cce/e32d7694-9c48-497a-b173-43968d858b60"
-					(reference "U8")
+					(reference "U9")
 					(unit 1)
 				)
@@
 		(dnp yes)
 		(fields_autoplaced yes)
-		(property "Reference" "R93"
+		(property "Reference" "R151"
 			(at 63.5 78.7399 90)
 			(effects
@@
 			(project "dashcam"
 				(path "/30d6913c-7aa4-4f56-9882-2ba08f7e2cce/e32d7694-9c48-497a-b173-43968d858b60"
-					(reference "R93")
+					(reference "R151")
 					(unit 1)
 				)
