File: hw/ethernet.kicad_sch (KiCad schematic)
At the start: 18 parts, among them J3 HR911130C, U1 AM6254ATCGHAALW, U6 RTL8211F-CG

Commit message: Ethernet...
Parts:
- removed C53, C54: CC0805KRX7R9BB104, pepy_sym_lib:[CAP_SMD_0805_2012Metric], symbol pepy_sym_lib:[CAP_SMD_0805_2012Metric]YAGEO CC0805KRX7R9BB104
- removed C55: CL21A475KAQNNNE, pepy_sym_lib:[CAP_SMD_0805_2012Metric], symbol pepy_sym_lib:[CAP_SMD_0805_2012Metric]Samsung Electro-Mechanics CL21A475KAQNNNE
- removed D5: TPD4E05U06DQAR, pepy_sym_lib:[ESD_PROT]Texas Instruments TPD4E05U06DQAR, symbol pepy_sym_lib:[ESD_PROT]Texas Instruments TPD4E05U06DQAR
- removed FB2: BLM18BD252SN1D, pepy_sym_lib:[FERRITE_BEAD_0603_1608Metric], symbol pepy_sym_lib:[FERRITE_BEAD]Murata Electronics BLM18PG121SN1D
- removed R65: 0805W8F2201T5E, pepy_sym_lib:[RES_SMD_0805_2012Metric], symbol pepy_sym_lib:[RES_SMD_0805_2012Metric]UNI-ROYAL(Uniroyal Elec) 0805W8F2201T5E
- added C193, C194: CC0201FRNPO9BN270, pepy_sym_lib:[CAP_SMD_0201_0603Metric], symbol pepy_sym_lib:[CAP_SMD_0201_0603Metric]YAGEO CC0201FRNPO9BN270
- added C196: CC0805KRX7R9BB104, pepy_sym_lib:[CAP_SMD_0805_2012Metric], symbol pepy_sym_lib:[CAP_SMD_0805_2012Metric]YAGEO CC0805KRX7R9BB104
- added C197, C198, C199, C200, C201, C203, C204, C205, C207: CC0201KRX5R6BB104, pepy_sym_lib:[CAP_SMD_0201_0603Metric], symbol pepy_sym_lib:[CAP_SMD_0201_0603Metric]YAGEO CC0201KRX5R6BB104
- added C202, C206, C53: CL03A105MQ3CSNH, pepy_sym_lib:[CAP_SMD_0201_0603Metric], symbol pepy_sym_lib:[CAP_SMD_0201_0603Metric]Samsung Electro-Mechanics CL03A105MQ3CSNH
- added C208, C54, C55: GRM035R60J475ME15D, pepy_sym_lib:[CAP_SMD_0201_0603Metric], symbol pepy_sym_lib:[CAP_SMD_0201_0603Metric]muRata GRM035R60J475ME15D
- added D31: TPD4E05U06DQAR, pepy_sym_lib:[ESD_PROT]Texas Instruments TPD4E05U06DQAR, symbol pepy_sym_lib:[ESD_PROT]Texas Instruments TPD4E05U06DQAR
- added L14: MHCD252012A-2R2M-A8S, pepy_sym_lib:[POWER_IND]Chilisin MHCD252012A-2R2M-A8S, symbol pepy_sym_lib:[POWER_IND]Chilisin MHCD252012A-2R2M-A8S
- added R149, R151, R65: 0402WGF0000TCE, pepy_sym_lib:[RES_SMD_0402_1005Metric], symbol pepy_sym_lib:[RES_SMD_0402_1005Metric]UNI-ROYAL(Uniroyal Elec) 0402WGF0000TCE
- added R150: 0402WGF2201TCE, pepy_sym_lib:[RES_SMD_0402_1005Metric], symbol pepy_sym_lib:[RES_SMD_0402_1005Metric]UNI-ROYAL(Uniroyal Elec) 0402WGF2201TCE
- added R152, R153, R154, R155, R156, R157, R158, R159, R160, R161, R162, R163, R164, R165, R166, R167, R168, R169: RC0201FR-074K7L, pepy_sym_lib:[RES_SMD_0201_0603Metric], symbol pepy_sym_lib:[RES_SMD_0201_0603Metric]YAGEO RC0201FR-074K7L
- added TP18: TestPoint, pepy_sym_lib:[TEST_POINT]TestPoint_Pad_D1.0mm, symbol pepy_sym_lib:[TEST_POINT]TestPoint
- added X3: X322525MRB4SI, pepy_sym_lib:[Crystal]YXC Crystal Oscillators X322525MRB4SI, symbol pepy_sym_lib:[Crystal]YXC Crystal Oscillators X322525MRB4SI
- D6: Manufacturer (none) -> TI; Package (none) -> USON-10(1x2.5)
- J3: Manufacturer (none) -> HANRUN(Zhongshan HanRun Elec)
- R66, R67, R69, R70, R71, R72: Nvalue 33 -> 33R; Tolerance (none) -> 1%
- R68: Tolerance (none) -> 1%
Connections:
- net GND: now also J3.10 (CHS_GND), C193.1, C194.2, C196.2, C197.1, C198.1, C199.1, C200.1, C201.1, C202.1, C203.1, C204.1, C205.1, C206.1, C207.1, C208.1, C53.1, C54.1, C55.1, D31.3 (GND), D31.8 (GND), R151.1, R153.1, R154.1, R156.1, R158.1, R159.1, R160.1, R164.1, R165.1, R166.1, X3.2 (GND), X3.4 (GND)
- net MDIO0_MDIO: now also R150.1; no longer U6.13 (MDC)
- net RGMII1_RD0: now also R156.2, R157.1
- net RGMII1_RD1: now also R154.2, R155.1
- net RGMII1_RD2: now also R152.1, R153.2
- net RGMII1_RD3: now also R158.2, R161.1
- net RGMII1_RXC: now also R159.2, R162.1
- net RGMII1_RX_CTL: now also U6.19 (TXCTL)
- net RGMII1_TD0: no longer R66.2
- net RGMII1_TD1: no longer R67.2
- net RGMII1_TD2: no longer R69.2
- net RGMII1_TD3: no longer R70.2
- net RGMII1_TXC: no longer R71.2
- net VDD_1V8: now also R150.2, R65.2
- net VDD_3V3: now also U6.11 (AVDD33), U6.29 (DVDD33), U6.40 (AVDD33), C199.2, C205.2, C206.2, C54.2, R167.2, R168.2, R169.2
- net at R69.1: no longer U1.AE18 (RGMII1_TD2)
- net at U1.AD18 (RGMII1_TD3): no longer R70.1
- net at U1.AD19 (RMII1_TX_CTL): no longer R72.1
- net at U1.AD20 (RGMII1_TD1): no longer R67.1
- net at U1.AE19 (RGMII1_TXC): no longer R71.1
- net at U1.AE20 (RGMII1_TD0): no longer R66.1
- net at U6.1 (MDIP0): now also D31.1 (D1+); no longer J3.2 (MDI0+)
- net at U6.2 (MDIN0): now also D31.2 (D1-); no longer J3.3 (MDI0-)
- net at U6.4 (MDIP1): now also D31.4 (D2+); no longer J3.4 (MDI1+)
- net at U6.5 (MDIN1): now also D31.5 (D2-); no longer J3.7 (MDI1-)
- net at J3.1 (CT): now also C196.1
- net at U6.12 (PHYRSTB): now also C197.2
- net PHY_VDD_1V0: now reaches U6.21 (DVDD10)
- net PHY_VDD_1V0: now also U6.3 (AVDD10), U6.38 (AVDD10), U6.8 (AVDD10), C198.2, C200.2, C201.2, C202.2, C203.2, C204.2, C53.2, C55.2, L14.2
- net PHY_VDDIO: now reaches U6.28 (DVDD_RG)
- net PHY_VDDIO: now also C207.2, C208.2, R152.2, R155.2, R157.2, R161.2, R162.2, R163.2, R65.1
- net at U6.30 (REG_OUT/LDO_OUT): now also L14.1
- net INTB: now reaches U6.31 (INTB/PMEB)
- net at U6.35 (CLKOUT): now also TP18.1
- net XI: now reaches U6.36 (XTAL_IN)
- net XI: now also C194.1, R151.2, X3.3 (X2)
- net at U6.37 (XTAL_OUT/EXT_CLK): now also R149.2
- net RGMII1_TX_CTL: no longer names the net of R72.2
- net RGMII1_TX_CTL: no longer U6.19 (TXCTL)
- new net: D6.5 (D2-), U6.10 (MDIN3)
- new net: D6.1 (D1+), U6.6 (MDIP2)
- new net: D6.2 (D1-), U6.7 (MDIN2)
- new net: D6.4 (D2+), U6.9 (MDIP3)
- new net LED0/CFG_EXT: R164.2, R167.1
- new net LED1/CFG_LDO0: R165.2, R168.1
- new net LED2/CFG_LDO1: R166.2, R169.1
- new net MCU_OBSCLK0: C193.2, R149.1, X3.1 (X1)
- new net MDI0+: D31.10 (NC), J3.2 (MDI0+)
- new net MDI0-: D31.9 (NC), J3.3 (MDI0-)
- new net MDI1+: D31.7 (NC), J3.4 (MDI1+)
- new net MDI1-: D31.6 (NC), J3.7 (MDI1-)
- new net MDI2+: D6.10 (NC), J3.5 (MDI2+)
- new net MDI2-: D6.9 (NC), J3.6 (MDI2-)
- new net MDI3+: D6.7 (NC), J3.8 (MDI3+)
- new net MDI3-: D6.6 (NC), J3.9 (MDI3-)
- new net MDIO0_MDC: U6.13 (MDC)
- new net RXCTL/PHYAD2: R160.2, R163.1
Other:
- note added: "100 ohms differential trace impedance."
- note added: "CFG_EXT = 0, CFG_LDO[1:0] = 10 : Internal 1.8V PHY AD[2:0] = 000: PHY Addr 000 PHY PLLOF = 0 : Enable PLL PHY TXDLY = 0 : TX delay: 0ns PHY RXDLY = 1 : RX delay: 2ns"
- note added: "Note: 1. If an external clock source is used, XO should be left floating.TR1_TAP1 2. For a 3.3-V clock source, a capacitor divider is recommended, the CD1 and CD2 capacitors used are recommended to be 27 pF."
- note added: "TO BE SET"
- note added: "The switching regulator 1.0V output pin (REG_OUT) should be connected only to DVDD10 and AVDD10 (do not provide this power source to other devices)."
- note added: "do i need ferrite beads here?"
- moved on the sheet: D6, R70, R73

Commit message: WIP SIM module
Parts:
- removed R149: 0402WGF0000TCE, pepy_sym_lib:[RES_SMD_0402_1005Metric], symbol pepy_sym_lib:[RES_SMD_0402_1005Metric]UNI-ROYAL(Uniroyal Elec) 0402WGF0000TCE
- added C127, C128, C146, C147: CC0201KRX5R6BB104, pepy_sym_lib:[CAP_SMD_0201_0603Metric], symbol pepy_sym_lib:[CAP_SMD_0201_0603Metric]YAGEO CC0201KRX5R6BB104
- added C149: CC1206KKX7RDBB102, pepy_sym_lib:[CAP_SMD_1206_3216Metric], symbol pepy_sym_lib:[CAP_SMD_1206_3216Metric]YAGEO CC1206KKX7RDBB102
- added D5, D6, D7: RB520S30T1G, pepy_sym_lib:[SCHOTTKY_DIODE]onsemi RB520S30T1G, symbol pepy_sym_lib:[SCHOTTKY_DIODE]onsemi RB520S30T1G
- added Q3, Q4: DMG1012T-7, pepy_sym_lib:[NMOS]DIODES DMG1012T-7, symbol pepy_sym_lib:[NMOS]DIODES DMG1012T-7
- added R101, R102, R93, R98: 0201WMF1002TEE, pepy_sym_lib:[RES_SMD_0201_0603Metric], symbol pepy_sym_lib:[RES_SMD_0201_0603Metric]UNI-ROYAL(Uniroyal Elec) 0201WMF1002TEE
- added R103, R104, R107, R83, R84, R86, R94, R95: 0402WGF0000TCE, pepy_sym_lib:[RES_SMD_0402_1005Metric], symbol pepy_sym_lib:[RES_SMD_0402_1005Metric]UNI-ROYAL(Uniroyal Elec) 0402WGF0000TCE
- added R105, R106: RC0402FR-071KL, pepy_sym_lib:[RES_SMD_0402_1005Metric], symbol pepy_sym_lib:[RES_SMD_0402_1005Metric]YAGEO RC0402FR-071KL
- added R77, R78, R79, R80, R81, R82, R91: RC0201FR-0733RL, pepy_sym_lib:[RES_SMD_0201_0603Metric], symbol pepy_sym_lib:[RES_SMD_0201_0603Metric]YAGEO RC0201FR-0733RL
- R108: renamed from R73; Tolerance (none) -> 1%
- renumbered C194 to C129, C193 to C130, C199 to C131, C198 to C132, C197 to C133, C54 to C134, C53 to C135, C205 to C136, C206 to C137, C204 to C138, C203 to C139, C201 to C140, C207 to C141, C200 to C142, C202 to C143, C208 to C144, C55 to C145, C196 to C148, D31 to D8, D6 to D9, J3 to J4, L14 to L8, R72 to R100, R153 to R109, R154 to R110, R156 to R111, R158 to R112, R159 to R113, R160 to R114, R164 to R115, R165 to R116, R166 to R117, R152 to R118, R155 to R119, R157 to R120, R161 to R121, R162 to R122, R163 to R123, R167 to R124, R168 to R125, R169 to R126, R150 to R85, R151 to R87, R66 to R88, R67 to R89, R68 to R90, R69 to R92, R65 to R96, R70 to R97, R71 to R99, TP18 to TP13, X3 to X2
Connections:
- net Earth is gone; now on net Earth_GBE: R108.1
- net LED0/CFG_EXT is gone; now on net LED0: R115.2, R124.1
- net LED1/CFG_LDO0 is gone; now on net LED1: R116.2, R125.1
- net LED2/CFG_LDO1 is gone; now on net LED2: R117.2, R126.1
- net GND: now also C127.1, C128.1, C146.1, C147.1, C149.2
- net INTB: now also Q4.3 (D), R102.1
- net MCU_OBSCLK0: now also R86.1; no longer C130.2, X2.1 (X1)
- net PHY_VDD_1V0: now also C128.2, C146.2, R84.1, R95.2; no longer C132.2, C135.2, C138.2, C139.2, C140.2, C143.2, U6.21 (DVDD10), U6.3 (AVDD10), U6.38 (AVDD10), U6.8 (AVDD10)
- net RGMII1_RD0: now also R77.1; no longer R111.2, R120.1, U6.25 (RXDLY/RXD0)
- net RGMII1_RD1: now also R80.1; no longer R110.2, R119.1, U6.24 (TXDLY/RXD1)
- net RGMII1_RD2: now also R78.1; no longer R109.2, R118.1, U6.23 (PLLOFF/RXD2)
- net RGMII1_RD3: now also R81.1; no longer R112.2, R121.1, U6.22 (PHYAD0/RXD3)
- net RGMII1_RXC: now also R79.1; no longer R113.2, R122.1, U6.27 (PHYAD1/RXC)
- net RGMII1_RX_CTL: now also R82.1; no longer U6.19 (TXCTL), U6.26 (PHYAD2/RXCTL)
- net RGMII1_TD0: now also R88.2
- net RGMII1_TD1: now also R89.2
- net RGMII1_TD2: now also R92.2
- net RGMII1_TD3: now also R97.2
- net RGMII1_TXC: now also R99.2
- net VDD_1V8: now also Q3.1 (G), Q4.1 (G), R101.2, R93.2
- net VDD_3V3: now also C127.2, C147.2, R83.1, R94.2; no longer C131.2, C134.2, C136.2, C137.2, R124.2, R125.2, R126.2, U6.11 (AVDD33), U6.29 (DVDD33), U6.40 (AVDD33)
- net at R92.1: now also U1.AE18 (RGMII1_TD2)
- net at TP13.1: now also R91.2; no longer U6.35 (CLKOUT)
- net at U1.AD18 (RGMII1_TD3): now also R97.1
- net at U1.AD19 (RMII1_TX_CTL): now also R100.1
- net at U1.AD20 (RGMII1_TD1): now also R89.1
- net at U1.AE19 (RGMII1_TXC): now also R99.1
- net at U1.AE20 (RGMII1_TD0): now also R88.1
- net at J4.11 (GELA): now also R104.1, R107.1
- net at J4.12 (GELC): now also R106.1
- net at J4.13 (YELC): now also R105.1
- net at J4.14 (YELA): now also R103.1
- net Earth_GBE: now reaches J4.15 (SHIELD)
- net Earth_GBE: now also J4.16 (SHIELD), C149.1
- net PHYRSTB: now reaches C133.2, U6.12 (PHYRSTB)
- net PHYRSTB: now also Q3.3 (D), R98.1
- net RGMII1_TX_CTL: now reaches R100.2
- net RGMII1_TX_CTL: now also U6.19 (TXCTL), U6.26 (PHYAD2/RXCTL), R82.2
- net XO: now reaches U6.37 (XTAL_OUT/EXT_CLK)
- net XO: now also C130.2, X2.1 (X1), R86.2
- net LED0: now reaches U6.32 (CFG_EXT/LED0)
- net LED0: now also R104.2
- net LED1: now reaches U6.33 (CFG_LDO0/LED1)
- net LED1: now also R106.2
- net LED2: now reaches U6.34 (CFG_LDO1/LED2)
- net LED2: now also R105.2
- new net: D5.2 (A), D6.2 (A), D7.2 (A), Q3.2 (S), R93.1
- new net: C138.2, C139.2, C140.2, C143.2, R95.1, U6.3 (AVDD10), U6.38 (AVDD10), U6.8 (AVDD10)
- new net: C132.2, C135.2, R84.2, U6.21 (DVDD10)
- new net: C136.2, C137.2, R94.1, U6.11 (AVDD33), U6.40 (AVDD33)
- new net: R91.1, U6.35 (CLKOUT)
- new net GBE_INTn: Q4.2 (S), R101.1
- new net GBE_RSTn: D5.1 (C)
- new net PHY_DVDD3V3: C131.2, C134.2, R102.2, R103.2, R107.2, R124.2, R125.2, R126.2, R83.2, R98.2, U6.29 (DVDD33)
- new net PORz_OUT: D6.1 (C)
- new net RESETSTATz: D7.1 (C)
- new net RXC/PHYAD1: R113.2, R122.1, R79.2, U6.27 (PHYAD1/RXC)
- new net RXD0/RXDLY: R111.2, R120.1, R77.2, U6.25 (RXDLY/RXD0)
- new net RXD1/TXDLY: R110.2, R119.1, R80.2, U6.24 (TXDLY/RXD1)
- new net RXD2/PLLOFF: R109.2, R118.1, R78.2, U6.23 (PLLOFF/RXD2)
- new net RXD3/PHYAD0: R112.2, R121.1, R81.2, U6.22 (PHYAD0/RXD3)
Other:
- note added: "1000M Link and Active (Transmitting or Receiving)"
- note added: "Gigabit Ethernet Interrupt AM62 pin: GPMC0_CSN1 (probably GPIO042?)"
- note added: "Gigabit Ethernet Reset AM62 pin: GPMC0_AD0 (probably GPIO015?)"
- note added: "Main Domain warm reset status output AM62 pin: F22 - RESESTATz"
- note added: "Power-On Reset output from the MCU AM62 pin: E21 - PORZ_OUT (cannot be disconnected by 0R)"
- note added: "Pull up for MDI0"
- note added: "Starp parallel resistors must be connected to HW CFG pins directly and not after the series termination resistors to avoid signal attenuation."
- note added: "TO MAC"
- note added: "When CFG_EXT(strapping pins) is pulled high this external source gets connected through a 0R resistor. DVDD_RG is an I/O pad, internal voltage appears on PHY_VDDIO."
- note removed: "2kV Cap"
- note removed: "Place resistors close to IC"
- note removed: "do i need ferrite beads here?"
- moved on the sheet: C136, C137, R100, R108, R109, R110, R111, R112, R113, R114, R115, R116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
