File: hw/pmic.kicad_sch (KiCad schematic)
At the start: 34 parts, among them U4 TPS6521907RHBR

Commit message: WIP SIM module
Parts:
- renumbered C36 to C110, C37 to C111, C38 to C112, C39 to C113, C40 to C114, C41 to C115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
