File: hw/sd.kicad_sch (KiCad schematic)
At the start: 27 parts, among them U1 AM6254ATCGHAALW, U7 TPS22918DBVR

Commit message: eMMC draft
Parts:
- added D17, D18, D19: RB520S30T1G, pepy_sym_lib:[SCHOTTKY_DIODE]onsemi RB520S30T1G, symbol pepy_sym_lib:[SCHOTTKY_DIODE]onsemi RB520S30T1G
- added R100, R101, R102, R103, R104, R108, R96, R97, R98, R99: RC0402FR-0749K9L, pepy_sym_lib:[RES_SMD_0402_1005Metric], symbol pepy_sym_lib:[RES_SMD_0402_1005Metric]YAGEO RC0402FR-0749K9L
- added R105: 0402WGF0000TCE, pepy_sym_lib:[RES_SMD_0402_1005Metric], symbol pepy_sym_lib:[RES_SMD_0402_1005Metric]UNI-ROYAL(Uniroyal Elec) 0402WGF0000TCE
- added R106, R107: 0201WMF1002TEE, pepy_sym_lib:[RES_SMD_0201_0603Metric], symbol pepy_sym_lib:[RES_SMD_0201_0603Metric]UNI-ROYAL(Uniroyal Elec) 0201WMF1002TEE
- added TP13: TestPoint, pepy_sym_lib:[TEST_POINT]TestPoint_Pad_D1.0mm, symbol pepy_sym_lib:[TEST_POINT]TestPoint
- added U10: KLMAG1JETD-B041, pepy_sym_lib:[eMMC]SAMSUNG KLMAG1JETD-B041, symbol pepy_sym_lib:[eMMC]SAMSUNG KLMAG1JETD-B041
Connections:
- net GND: now also R107.1, R108.1, U10.A6 (VSS), U10.C4 (VSS), U10.E7 (VSS), U10.G5 (VSS), U10.H10 (VSS), U10.J5 (VSS), U10.K8 (VSS), U10.N2 (VSS), U10.N5 (VSS), U10.P4 (VSS), U10.P6 (VSS)
- net RESETSTATz: now also D17.1 (C)
- net at U1.AA1 (MMC0_DAT1): now also R102.1, U10.A4 (DAT1)
- net at U1.AA2 (MMC0_DAT0): now also R103.1, U10.A3 (DAT0)
- net at U1.AA3 (MMC0_DAT2): now also R101.1, U10.A5 (DAT2)
- net at U1.AB1 (MMC0_CLK): now also R105.1
- net at U1.AB2 (MMC0_DAT4): now also R99.1, U10.B3 (DAT4)
- net at U1.AC1 (MMC0_DAT5): now also R98.1, U10.B4 (DAT5)
- net at U1.AC2 (MMC0_DAT7): now also R96.1, U10.B6 (DAT7)
- net at U1.AD2 (MMC0_DAT6): now also R97.1, U10.B5 (DAT6)
- net at U1.Y3 (MMC0_CMD): now also R104.1, U10.M5 (CMD)
- net at U1.Y4 (MMC0_DAT3): now also R100.1, U10.B2 (DAT3)
- new net: D17.2 (A), D18.2 (A), D19.2 (A), R106.1, U10.K5 (RST_N)
- new net: R107.2, TP13.1, U10.H5 (DS)
- new net: R105.2, R108.2, U10.M6 (CLK)
- new net PORz_OUT: D19.1 (C)
- new net VDD_1V8: R100.2, R101.2, R102.2, R103.2, R104.2, R106.2, R96.2, R97.2, R98.2, R99.2
- new net eMMC_RSTn: D18.1 (C)
Other:
- note added: "For dumping reasons: 22 Ohm?"
- note added: "SD"
- note added: "eMMC"
- moved on the sheet: R82, R83, U1G

Commit message: WIP SIM module
Parts:
- renumbered C56 to C150, C57 to C151, C58 to C152, C59 to C153, C60 to C154, D7 to D10, D8 to D11, D9 to D12, D10 to D13, D11 to D14, D12 to D15, D17 to D16, D18 to D17, D19 to D18, D13 to D19, D14 to D20, D15 to D21, R82 to R127, R105 to R128, R83 to R129, R74 to R130, R96 to R131, R97 to R132, R98 to R133, R99 to R134, R108 to R135, R100 to R136, R75 to R137, R101 to R138, R76 to R139, R102 to R140, R78 to R141, R103 to R142, R77 to R143, R104 to R144, R79 to R145, R106 to R146, R80 to R147, R107 to R148, R81 to R149, TP13 to TP14, U10 to U8
