File: hw/soc_power_sch.kicad_sch (KiCad schematic)
At the start: 1 part, among them U1 AM6254ATCGHAALW

Commit message: Ethernet...
Parts:
- added C67, C71, C75, C78, C81, C84, C86, C88, C89, C91, C94, C97: CC0201KRX5R6BB104, pepy_sym_lib:[CAP_SMD_0201_0603Metric], symbol pepy_sym_lib:[CAP_SMD_0201_0603Metric]YAGEO CC0201KRX5R6BB104
- added C68, C72, C76, C79, C82, C85, C87, C92, C95, C98: GRM033R71A103KA01D, pepy_sym_lib:[CAP_SMD_0201_0603Metric], symbol pepy_sym_lib:[CAP_SMD_0201_0603Metric]muRata GRM033R71A103KA01D
- added C69, C70, C90, C93, C96: GRM035R60J475ME15D, pepy_sym_lib:[CAP_SMD_0201_0603Metric], symbol pepy_sym_lib:[CAP_SMD_0201_0603Metric]muRata GRM035R60J475ME15D
- added C73, C74, C77, C80, C83: CL03A105MQ3CSNH, pepy_sym_lib:[CAP_SMD_0201_0603Metric], symbol pepy_sym_lib:[CAP_SMD_0201_0603Metric]Samsung Electro-Mechanics CL03A105MQ3CSNH
- added H1: X6511WV-02H-C30D60, pepy_sym_lib:[2x1_PIN_HEADER_STR]XKB Connection X6511WV-02H-C60D30, symbol pepy_sym_lib:[2x1_PIN_HEADER_STR]XKB Connection X6511WV-02H-C60D30
- added R109: 0402WGF1102TCE, pepy_sym_lib:[RES_SMD_0402_1005Metric], symbol pepy_sym_lib:[RES_SMD_0402_1005Metric]UNI-ROYAL 0402WGF1102TCE
- added R110: RC0402FR-07100KL, pepy_sym_lib:[RES_SMD_0402_1005Metric], symbol pepy_sym_lib:[RES_SMD_0402_1005Metric]YAGEO RC0402FR-07100KL
- added R111: 0201WMF1002TEE, pepy_sym_lib:[RES_SMD_0201_0603Metric], symbol pepy_sym_lib:[RES_SMD_0201_0603Metric]UNI-ROYAL(Uniroyal Elec) 0201WMF1002TEE
Connections:
- net VDD_CORE: now also U1.F8 (VDD_CANUART), U1.W12 (VDDA_CORE_USB), U1.W13 (VDDA_CORE_CSIRX0), C90.2, C91.2, C92.2, C93.2, C94.2, C95.2, C96.2, C97.2, C98.2
- net VDD_1V8: now reaches U1.F11 (VDDSHV_MCU)
- net VDD_1V8: now also U1.G10 (VMON_1P8_SOC), U1.G12 (VDDSHV_MCU), U1.J18 (VDDSHV6), U1.N18 (VDDSHV3), U1.P18 (VDDSHV3), U1.T19 (VDDSHV3), U1.T7 (VDDSHV4), U1.U18 (VDDSHV3), U1.W16 (VDDSHV2), U1.W19 (VDDSHV2), H1.2
- net VDD_3V3: now reaches U1.F15 (VDDSHV0)
- net VDD_3V3: now also U1.G14 (VDDSHV0), U1.H9 (VDDSHV_CANUART), U1.K10 (VMON_3P3_SOC), U1.L18 (VDDSHV1), U1.M19 (VDDSHV1), U1.Y13 (VDDA_3P3_USB)
- net VDDA_1V8: now reaches U1.G16 (VDDA_TEMP1)
- net VDDA_1V8: now also U1.G17 (VDDSHV5), U1.G7 (VDDS_OSC0), U1.L11 (VDDA_MCU), U1.L14 (VDD_PLL2), U1.T9 (VDDA_TEMP0), U1.U11 (VDD_PLL0), U1.U15 (VDD_PLL1), U1.W10 (VDDA_1P8_OLDI1), U1.W14 (VDDA_1P8_CSIRX0), U1.W9 (VDDA_1P8_OLDI0), U1.Y11 (VDDA_1P8_USB), C67.2, C68.2, C69.2, C70.2, C71.2, C72.2, C73.2, C74.2, C75.2, C76.2, C77.2, C78.2, C79.2, C80.2, C81.2, C82.2, C83.2, C84.2, C85.2, C86.2, C87.2, C88.2, C89.2
- net VDDA_SYS_MON: now reaches U1.H10 (VMON_ER_VSYS)
- net VDDA_SYS_MON: now also R109.2, R110.1
- net VDDA_0V85: now reaches U1.J12 (VDDR_CORE)
- net VDDA_0V85: now also U1.K16 (VDDR_CORE), U1.N12 (VDDR_CORE), U1.N14 (VDDR_CORE), U1.P16 (VDDR_CORE), U1.R12 (VDDR_CORE), U1.T10 (VDDR_CORE), U1.U14 (VDDR_CORE)
- net at U1.J8 (VPP): now also H1.1, R111.2
- net VDD_1V2: now reaches U1.K9 (VDDS_DDR)
- net VDD_1V2: now also U1.L8 (VDDS_DDR), U1.M9 (VDDS_DDR_C), U1.P9 (VDDS_DDR), U1.R8 (VDDS_DDR)
- new net GND: C67.1, C68.1, C69.1, C70.1, C71.1, C72.1, C73.1, C74.1, C75.1, C76.1, C77.1, C78.1, C79.1, C80.1, C81.1, C82.1, C83.1, C84.1, C85.1, C86.1, C87.1, C88.1, C89.1, C90.1, C91.1, C92.1, C93.1, C94.1, C95.1, C96.1, C97.1, C98.1, R109.1, R111.1
- new net VSYS_5V: R110.2

Commit message: WIP SIM module
Parts:
- renumbered C82 to C100, C90 to C101, C93 to C102, C96 to C103, C91 to C104, C94 to C105, C97 to C106, C92 to C107, C95 to C108, C98 to C109, C88 to C78, C69 to C79, C70 to C80, C67 to C81, C86 to C82, C68 to C83, C87 to C84, C89 to C85, C73 to C86, C83 to C87, C71 to C88, C84 to C89, C72 to C90, C85 to C91, C74 to C92, C77 to C93, C80 to C94, C75 to C95, C78 to C96, C81 to C97, C76 to C98, C79 to C99, R110 to R63, R109 to R64, R111 to R65
