File: hw/usb_c.kicad_sch (KiCad schematic)
At the start: 12 parts, among them J1 TYPE-C 16PIN 2MD(073), U1 AM6254ATCGHAALW, U3 TVS0500DRVR

Commit message: WIP SIM module
Parts:
- renumbered J1 to J2, L2 to L4, R6 to R15, R7 to R16, R8 to R17, R9 to R18, R10 to R19, R11 to R20
Changed lines of the file:
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@@
 		(dnp no)
 		(fields_autoplaced yes)
-		(property "Reference" "R10"
+		(property "Reference" "R19"
 			(at 175.26 62.23 0)
 			(effects
@@
 			(project "dashcam"
 				(path "/30d6913c-7aa4-4f56-9882-2ba08f7e2cce/c5ef26fc-2066-490b-8721-1c4a1c83f953"
-					(reference "R10")
+					(reference "R19")
 					(unit 1)
 				)
@@
 		(on_board yes)
 		(dnp no)
-		(property "Reference" "#PWR07"
+		(property "Reference" "#PWR011"
 			(at 33.02 77.47 0)
 			(effects
@@
 			(project "dashcam"
 				(path "/30d6913c-7aa4-4f56-9882-2ba08f7e2cce/c5ef26fc-2066-490b-8721-1c4a1c83f953"
-					(reference "#PWR07")
+					(reference "#PWR011")
 					(unit 1)
 				)
@@
 		(dnp no)
 		(fields_autoplaced yes)
-		(property "Reference" "R7"
+		(property "Reference" "R16"
 			(at 33.02 105.4099 90)
 			(effects
@@
 			(project "dashcam"
 				(path "/30d6913c-7aa4-4f56-9882-2ba08f7e2cce/c5ef26fc-2066-490b-8721-1c4a1c83f953"
-					(reference "R7")
+					(reference "R16")
 					(unit 1)
 				)
@@
 		(dnp no)
 		(fields_autoplaced yes)
-		(property "Reference" "R8"
+		(property "Reference" "R17"
 			(at 154.94 53.3399 90)
 			(effects
@@
 			(project ""
 				(path "/30d6913c-7aa4-4f56-9882-2ba08f7e2cce/c5ef26fc-2066-490b-8721-1c4a1c83f953"
-					(reference "R8")
+					(reference "R17")
 					(unit 1)
 				)
@@
 		(dnp no)
 		(fields_autoplaced yes)
-		(property "Reference" "J1"
+		(property "Reference" "J2"
 			(at 57.785 69.85 0)
 			(effects
@@
 			(project ""
 				(path "/30d6913c-7aa4-4f56-9882-2ba08f7e2cce/c5ef26fc-2066-490b-8721-1c4a1c83f953"
-					(reference "J1")
+					(reference "J2")
 					(unit 1)
 				)
@@
 		(on_board yes)
 		(dnp no)
-		(property "Reference" "#PWR05"
+		(property "Reference" "#PWR09"
 			(at 24.13 102.87 0)
 			(effects
@@
 			(project "dashcam"
 				(path "/30d6913c-7aa4-4f56-9882-2ba08f7e2cce/c5ef26fc-2066-490b-8721-1c4a1c83f953"
-					(reference "#PWR05")
+					(reference "#PWR09")
 					(unit 1)
 				)
@@
 		(on_board yes)
 		(dnp no)
-		(property "Reference" "#PWR010"
+		(property "Reference" "#PWR014"
 			(at 92.71 101.6 0)
 			(effects
@@
 			(project "dashcam"
 				(path "/30d6913c-7aa4-4f56-9882-2ba08f7e2cce/c5ef26fc-2066-490b-8721-1c4a1c83f953"
-					(reference "#PWR010")
+					(reference "#PWR014")
 					(unit 1)
 				)
@@
 		(on_board yes)
 		(dnp no)
-		(property "Reference" "#PWR09"
+		(property "Reference" "#PWR013"
 			(at 50.8 62.23 0)
 			(effects
@@
 			(project ""
 				(path "/30d6913c-7aa4-4f56-9882-2ba08f7e2cce/c5ef26fc-2066-490b-8721-1c4a1c83f953"
-					(reference "#PWR09")
+					(reference "#PWR013")
 					(unit 1)
 				)
@@
 		(dnp no)
 		(fields_autoplaced yes)
-		(property "Reference" "R11"
+		(property "Reference" "R20"
 			(at 181.61 97.7899 90)
 			(effects
@@
 			(project ""
 				(path "/30d6913c-7aa4-4f56-9882-2ba08f7e2cce/c5ef26fc-2066-490b-8721-1c4a1c83f953"
-					(reference "R11")
+					(reference "R20")
 					(unit 1)
 				)
@@
 		(dnp no)
 		(fields_autoplaced yes)
-		(property "Reference" "L2"
+		(property "Reference" "L4"
 			(at 149.86 78.74 0)
 			(effects
@@
 			(project ""
 				(path "/30d6913c-7aa4-4f56-9882-2ba08f7e2cce/c5ef26fc-2066-490b-8721-1c4a1c83f953"
-					(reference "L2")
+					(reference "L4")
 					(unit 1)
 				)
@@
 		(on_board yes)
 		(dnp no)
-		(property "Reference" "#PWR06"
+		(property "Reference" "#PWR010"
 			(at 30.48 118.11 0)
 			(effects
@@
 			(project "dashcam"
 				(path "/30d6913c-7aa4-4f56-9882-2ba08f7e2cce/c5ef26fc-2066-490b-8721-1c4a1c83f953"
-					(reference "#PWR06")
+					(reference "#PWR010")
 					(unit 1)
 				)
@@
 		(on_board yes)
 		(dnp no)
-		(property "Reference" "#PWR08"
+		(property "Reference" "#PWR012"
 			(at 46.99 111.76 0)
 			(effects
@@
 			(project ""
 				(path "/30d6913c-7aa4-4f56-9882-2ba08f7e2cce/c5ef26fc-2066-490b-8721-1c4a1c83f953"
-					(reference "#PWR08")
+					(reference "#PWR012")
 					(unit 1)
 				)
@@
 		(dnp no)
 		(fields_autoplaced yes)
-		(property "Reference" "R9"
+		(property "Reference" "R18"
 			(at 154.94 63.4999 90)
 			(effects
@@
 			(project ""
 				(path "/30d6913c-7aa4-4f56-9882-2ba08f7e2cce/c5ef26fc-2066-490b-8721-1c4a1c83f953"
-					(reference "R9")
+					(reference "R18")
 					(unit 1)
 				)
@@
 		(dnp no)
 		(fields_autoplaced yes)
-		(property "Reference" "R6"
+		(property "Reference" "R15"
 			(at 26.67 90.1699 90)
 			(effects
@@
 			(project ""
 				(path "/30d6913c-7aa4-4f56-9882-2ba08f7e2cce/c5ef26fc-2066-490b-8721-1c4a1c83f953"
-					(reference "R6")
+					(reference "R15")
 					(unit 1)
 				)
@@
 		(on_board yes)
 		(dnp no)
-		(property "Reference" "#PWR013"
+		(property "Reference" "#PWR017"
 			(at 179.07 110.49 0)
 			(effects
@@
 			(project ""
 				(path "/30d6913c-7aa4-4f56-9882-2ba08f7e2cce/c5ef26fc-2066-490b-8721-1c4a1c83f953"
-					(reference "#PWR013")
+					(reference "#PWR017")
 					(unit 1)
 				)
@@
 		(on_board yes)
 		(dnp no)
-		(property "Reference" "#PWR012"
+		(property "Reference" "#PWR016"
 			(at 170.18 74.93 0)
 			(effects
@@
 			(project ""
 				(path "/30d6913c-7aa4-4f56-9882-2ba08f7e2cce/c5ef26fc-2066-490b-8721-1c4a1c83f953"
-					(reference "#PWR012")
+					(reference "#PWR016")
 					(unit 1)
 				)
@@
 		(on_board yes)
 		(dnp no)
-		(property "Reference" "#PWR011"
+		(property "Reference" "#PWR015"
 			(at 152.4 76.2 0)
 			(effects
@@
 			(project ""
 				(path "/30d6913c-7aa4-4f56-9882-2ba08f7e2cce/c5ef26fc-2066-490b-8721-1c4a1c83f953"
-					(reference "#PWR011")
+					(reference "#PWR015")
 					(unit 1)
 				)
